File: glassesBoard/glassesBoard.sch (EAGLE design)
At the start: 1 part

Commit message: Added input protection design
Parts:
- added C1, C2, C3, C4, C5, C6, C7: 1uF, thanics-capacitor:CL05A105MP5NNNC
- added D1: BAS40-06, glasses:BAS40-06SOT-23-3
- added F1: SF-0603S200-2, thanics-resistor:SF-0603S200-2
- added J1: AXK724147G, glasses:AXK724147G
- added J2: 105450-0101, 105450-0101:105450-0101
- added R1, R2: 10k, 10k-resistor(0603):RC0603JR-0710KLRC0603N-M
- added TP1, TP2, TP3: TPB2,54, testpad:TPB2,54
- added U$1: DART-SD410, glasses:DART-SD410
- added U$2: MICROSD, glasses:MICROSD
- added U2: APDS-9960, glasses:APDS-9960
- added U3: 1.8, glasses:MIC5504-1.8SOT23-5
- added U4: 3.3, glasses:MIC5504-3.3
- added U5, U6: SSM3J338RSOT-23F, glasses:SSM3J338RSOT-23F
- added U7: (no value), attiny10:ATTINY10-TSHR6ST1-M
- added U8: IQS263BDFN10, glasses:IQS263BDFN10
Connections:
- new net !TOUCH_INT: D1.C1, U8.RDY
- new net +1V8: C4.1, U3.VOUT
- new net +3V3: C5.1, R2.11, U4.VOUT, U7.VCC, U8.VDDHI
- new net BATT_CNTL: D1.C2
- new net FUSE_SNS: F1.2, R1.22, U6.S
- new net GND: C1.2, C2.2, C3.2, C4.2, C5.2, C7.2, U$2.VSS, U3.GND, U4.GND, U5.G
- new net MIPI_CSI0_CLK_N: U$1G$1.MIPI_CSI0_CLK_N
- new net MIPI_CSI0_CLK_P: U$1G$1.MIPI_CSI0_CLK_P
- new net MIPI_CSI0_DATA0_N: U$1G$1.MIPI_CSI0_DATA0_N
- new net MIPI_CSI0_DATA0_P: U$1G$1.MIPI_CSI0_DATA0_P
- new net MIPI_CSI0_DATA1_N: U$1G$1.MIPI_CSI0_DATA1_N
- new net MIPI_CSI0_DATA1_P: U$1G$1.MIPI_CSI0_DATA1_P
- new net MIPI_CSI0_DATA2_N: U$1G$1.MIPI_CSI0_DATA2_N
- new net MIPI_CSI0_DATA2_P: U$1G$1.MIPI_CSI0_DATA2_P
- new net MIPI_CSI0_DATA3_N: U$1G$1.MIPI_CSI0_DATA3_N
- new net MIPI_CSI0_DATA3_P: U$1G$1.MIPI_CSI0_DATA3_P
- new net MIPI_DSI0_CLK_N: U$1G$1.MIPI_DSI0_CLK_N
- new net MIPI_DSI0_CLK_P: U$1G$1.MIPI_DSI0_CLK_P
- new net MIPI_DSI0_DATA0_N: U$1G$1.MIPI_DSI0_DATA0_N
- new net MIPI_DSI0_DATA0_P: U$1G$1.MIPI_DSI0_DATA0_P
- new net MIPI_DSI0_DATA1_N: U$1G$1.MIPI_DSI0_DATA1_N
- new net MIPI_DSI0_DATA1_P: U$1G$1.MIPI_DSI0_DATA1_P
- new net MIPI_DSI0_DATA2_N: U$1G$1.MIPI_DSI0_DATA2_N
- new net MIPI_DSI0_DATA2_P: U$1G$1.MIPI_DSI0_DATA2_P
- new net MIPI_DSI0_DATA3_N: U$1G$1.MIPI_DSI0_DATA3_N
- new net MIPI_DSI0_DATA3_P: U$1G$1.MIPI_DSI0_DATA3_P
- new net N$2: F1.1, U5.S
- new net N$4: R2.22, TP1.TP, U7.PB3_(!RESET)
- new net N$5: TP3.TP, U7.(PCINT1/TPICLK)_PB1
- new net N$6: C7.1, D1.A, R1.11, U6.G
- new net N$7: TP2.TP, U7.(PCINT0/TPIDATA)_PB0
- new net P$1: C2.1, C3.1, U3.EN, U3.VIN, U4.EN, U4.VIN, U6.D
- new net SDC2_CLK: U$1G$1.SDC2_CLK, U$2.CLK
- new net SDC2_CMD: U$1G$1.SDC2_CMD, U$2.CMD
- new net SDC2_DATA_0: U$1G$1.SDC2_DATA_0, U$2.DAT0
- new net SDC2_DATA_1: U$1G$1.SDC2_DATA_1, U$2.DAT1
- new net SDC2_DATA_2: U$1G$1.SDC2_DATA_2, U$2.DAT2
- new net SDC2_DATA_3: U$1G$1.SDC2_DATA_3, U$2.CD/DAT3
- new net USB_HS_D_N: U$1G$2.USB_HS_D_N
- new net USB_HS_D_P: U$1G$2.USB_HS_D_P
- new net USB_HS_ID: U$1G$2.GPIO121
- new net VBATT_IN: U5.D
- new net VREG_L11_SDC: C1.1, U$1G$2.VREG_L11_SDC, U$1G$2.VREG_L11_SDC@1, U$2.VDD
Other:
- note added: "Input Protection: U5 - Reverse polarity protection for battery F1 - 2A fuse (blows at 5A within 5 sec) FUSE_SNS - ATTiny turns U6 OFF when ADC senses abnormal voltage drop across fuse F1"
- note added: "NEED TO FIX THIS"
- note added: "Power ON sequence: Touch Sensor reads button press, sends interrupt low, U6 turns ON. ATTiny latches U6 ON before Touch interrupt goes high"
- note added: "USB Mode ID: Low: Host Mode High: Device Mode"
- moved on the sheet: U1

Commit message: Added display converters and organized schematic
Parts:
- removed C7: 1uF, thanics-capacitor:CL05A105MP5NNNC
- removed D1: BAS40-06, glasses:BAS40-06SOT-23-3
- removed J2: 105450-0101, 105450-0101:105450-0101
- removed U2: APDS-9960, glasses:APDS-9960
- added C50: 22uF, thanics-capacitor:CL21A226MOCLRNC
- added C8, C9: 10uF, thanics-capacitor:GRM188R61A106KE69D
- added F2: SF-0603S200-2, thanics-resistor:SF-0603S200-2
- added J7: 105450-0101, 105450-0101:105450-0101
- added R3: 10k, thanics-resistor:RC0402JR-0710KL
- added R4: 2.15k, thanics-resistor:RC0402FR-072K15L
- added R5: 1k, thanics-resistor:RC0402FR-071KL
- added R6, R7: 3.2k, thanics-resistor:RT0402DRE073K2L
- added R8: 56k, thanics-resistor:RC0402JR-0756KL
- added U10: ATTINY20-MMH, attiny20:ATTINY20-MMH
- added U11: SN65LVDS822VQFN48, glasses:SN65LVDS822VQFN48
- R1: value 10k -> 56k; device 10k-resistor(0603):RC0603JR-0710KLRC0603N-M -> thanics-resistor:RC0402JR-0756KL
- R2: device 10k-resistor(0603):RC0603JR-0710KLRC0603N-M -> thanics-resistor:RC0402JR-0710KL
- U7: value (none) -> SN65DSI83PBGA-N64; device attiny10:ATTINY10-TSHR6ST1-M -> glasses:SN65DSI83PBGA-N64
Connections:
- removed net FUSE_SNS: F1.2, R1.22, U6.S
- removed net N$6: C7.1, D1.A, R1.11, U6.G
- new net !RST: R2.2, TP3.TP, U10.PB3
- new net !SHUTDOWN_INT: U10.PA3
- new net +5V: C6.1, C8.1, F2.2, R1.2, R2.1, R8.2, U10.VCC
- new net ADC: R5.1, R7.2, U10.PA0
- new net AIN1: R4.1, R6.2, U10.PA2
- new net FUSED_VBATT: C2.1, F1.2, R3.1, R4.2, R7.1, U3.EN, U3.VIN, U6.S
- new net I2C_SCL_5V: U10.PA7
- new net I2C_SDA_5V/TPIDATA: TP2.TP, U10.PB1
- new net N$1: U11.A0P, U7.A_Y0P
- new net N$10: U11.A3N, U7.A_Y3N
- new net N$11: U11.CLKP, U7.A_CLKP
- new net N$12: U11.CLKN, U7.A_CLKN
- new net N$3: U11.A0N, U7.A_Y0N
- new net N$50: J7.CC1, R8.1
- new net N$51: C50.1, F2.1, J7.VBUS@1, J7.VBUS@2, J7.VBUS@3, J7.VBUS@4
- new net N$63: J7.CC2, R1.1
- new net N$8: U11.A2N, U7.A_Y2N
- new net N$9: U11.A3P, U7.A_Y3P
- new net TPICLK: TP1.TP, U10.PB0
- net !TOUCH_INT: no longer D1.C1
- net +1V8: now also U10.PA1
- net +3V3: no longer R2.11, U7.VCC
- net BATT_CNTL: now also R3.2, U10.PA4, U6.G; no longer D1.C2
- net GND: now also C50.2, C6.2, C8.2, J7.GND@1, J7.GND@2, J7.GND@3, J7.GND@4, J7.SHIELD, R5.2, R6.1, U10.EPAD, U10.GND; no longer C7.2
- net MIPI_DSI0_CLK_N: now also U7.DACN
- net MIPI_DSI0_CLK_P: now also U7.DACP
- net MIPI_DSI0_DATA0_N: now also U7.DA0N
- net MIPI_DSI0_DATA0_P: now also U7.DA0P
- net MIPI_DSI0_DATA1_N: now also U7.DA1N
- net MIPI_DSI0_DATA1_P: now also U7.DA1P
- net MIPI_DSI0_DATA2_N: now also U7.DA2N
- net MIPI_DSI0_DATA2_P: now also U7.DA2P
- net MIPI_DSI0_DATA3_N: now also U7.DA3N
- net MIPI_DSI0_DATA3_P: now also U7.DA3P
- net N$4: now also U11.A1P, U7.A_Y1P; no longer R2.22, TP1.TP, U7.PB3_(!RESET)
- net N$5: now also U11.A1N, U7.A_Y1N; no longer TP3.TP, U7.(PCINT1/TPICLK)_PB1
- net N$7: now also U11.A2P, U7.A_Y2P; no longer TP2.TP, U7.(PCINT0/TPIDATA)_PB0
- net P$1: no longer C2.1, U3.EN, U3.VIN
- net USB_HS_D_N: now also J7.D-@1, J7.D-@2
- net USB_HS_D_P: now also J7.D+@1, J7.D+@2
Other:
- note added: "Camera"
- note added: "Display"
- note added: "Input/Power Management"
- note added: "Power Supplies"
- note added: "Sensors"
- note added: "Snapdragon 410E SoM"
- note added: "USB C/microSD"
- note removed: "NEED TO FIX THIS"
- moved on the sheet: C1, C2, C3, C4, C5, C6, F1, J1, TP1, TP2, TP3, U$2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

Commit message: Added boot select circuitry
Parts:
- added C7: 22uF, thanics-capacitor:CL21A226MOCLRNC
- added L1: 4.7uH, glasses:DFE252012P-4R7M=P2"
- added R10, R11, R14, R15, R16, R9: 10k, thanics-resistor:RC0402JR-0710KL
- added R12, R13: 5.1k, thanics-resistor:RMCF0603JT5K10
- added U12: NLAS2750, glasses:NLAS2750
- added U13, U15, U9: NX3020NAK, glasses:NX3020NAK
- added U14: SSM3J338RSOT-23F, glasses:SSM3J338RSOT-23F
- added U2: TPS613222A, glasses:TPS613222A
- C9: value 10uF -> 22uF; device thanics-capacitor:GRM188R61A106KE69D -> thanics-capacitor:CL21A226MOCLRNC
Connections:
- removed net MIPI_CSI0_CLK_N: U$1G$1.MIPI_CSI0_CLK_N
- removed net MIPI_CSI0_CLK_P: U$1G$1.MIPI_CSI0_CLK_P
- removed net MIPI_CSI0_DATA0_N: U$1G$1.MIPI_CSI0_DATA0_N
- removed net MIPI_CSI0_DATA0_P: U$1G$1.MIPI_CSI0_DATA0_P
- removed net MIPI_CSI0_DATA1_N: U$1G$1.MIPI_CSI0_DATA1_N
- removed net MIPI_CSI0_DATA1_P: U$1G$1.MIPI_CSI0_DATA1_P
- removed net MIPI_CSI0_DATA2_N: U$1G$1.MIPI_CSI0_DATA2_N
- removed net MIPI_CSI0_DATA2_P: U$1G$1.MIPI_CSI0_DATA2_P
- removed net MIPI_CSI0_DATA3_N: U$1G$1.MIPI_CSI0_DATA3_N
- removed net MIPI_CSI0_DATA3_P: U$1G$1.MIPI_CSI0_DATA3_P
- removed net N$50: J7.CC1, R8.1
- removed net N$63: J7.CC2, R1.1
- new net BOOT_CONFIG_0: U$1G$2.GPIO80
- new net BOOT_CONFIG_1: U$1G$2.GPIO81
- new net BOOT_CONFIG_2: U$1G$2.GPIO82
- new net BOOT_CONFIG_3: U$1G$2.GPIO83
- new net BOOT_CONFIG_5: R10.1, U$1G$2.GPIO86
- new net FORCED_USB_BOOT: U$1G$1.GPIO37
- new net I2C0_SCL: U$1G$1.GPIO7
- new net I2C0_SDA: U$1G$1.GPIO6
- new net I2C2_SCL: U$1G$1.GPIO30
- new net I2C2_SDA: U$1G$1.GPIO29
- new net I2C3_SCL: U$1G$2.GPIO15
- new net I2C3_SDA: U$1G$2.GPIO14
- new net MIPI_CSI1_CLK_N: U$1G$1.MIPI_CSI1_CLK_N
- new net MIPI_CSI1_CLK_P: U$1G$1.MIPI_CSI1_CLK_P
- new net MIPI_CSI1_DATA0_N: U$1G$1.MIPI_CSI1_DATA0_N
- new net MIPI_CSI1_DATA0_P: U$1G$1.MIPI_CSI1_DATA0_P
- new net MIPI_CSI1_DATA1_N: U$1G$1.MIPI_CSI1_DATA1_N
- new net MIPI_CSI1_DATA1_P: U$1G$1.MIPI_CSI1_DATA1_P
- new net N$13: U10.PA6, U9.G
- new net N$14: R11.1
- new net N$15: R14.1
- new net N$16: J7.CC2, U12.COM2
- new net N$17: J7.CC1, U12.COM1
- new net N$18: R13.2, U12.NO2
- new net N$19: R12.2, U12.NO1
- new net N$20: R1.1, U12.NC1
- new net N$21: R8.1, U12.NC2
- new net N$22: R15.2, U12.IN1, U12.IN2, U13.S
- new net N$23: R16.1, U14.G, U15.D
- new net N$6: L1.1, U2.SW
- new net PHONE_ON_N: R9.1, U$1G$2.PHONE_ON_N, U9.D
- net +1V8: now also R10.2, R11.2, R14.2, R9.2
- net +5V: now also R16.2, U12.VCC, U13.D, U14.S, U2.VOUT
- net AIN1: now also R6.1; no longer R6.2
- net FUSED_VBATT: now also L1.2
- net GND: now also C7.1, C9.2, R12.1, R13.1, R15.1, R6.2, U$1G$1.DGND, U$1G$1.DGND@1, U$1G$1.DGND@10, U$1G$1.DGND@11, U$1G$1.DGND@2, U$1G$1.DGND@3, U$1G$1.DGND@4, U$1G$1.DGND@5, U$1G$1.DGND@6, U$1G$1.DGND@7, U$1G$1.DGND@8, U$1G$1.DGND@9, U$1G$1.GND_CFILT, U$1G$1.GND_CFILT@1, U$1G$2.DGND, U$1G$2.DGND@1, U$1G$2.DGND@10, U$1G$2.DGND@11, U$1G$2.DGND@12, U$1G$2.DGND@13, U$1G$2.DGND@14, U$1G$2.DGND@15, U$1G$2.DGND@16, U$1G$2.DGND@2, U$1G$2.DGND@3, U$1G$2.DGND@4, U$1G$2.DGND@5, U$1G$2.DGND@6, U$1G$2.DGND@7, U$1G$2.DGND@8, U$1G$2.DGND@9, U12.GND, U15.S, U2.GND, U9.S; no longer R6.1
- net P$1: now also C7.2, C9.1, U$1G$1.VPH_POWER, U$1G$1.VPH_POWER@1, U$1G$1.VPH_POWER@2, U$1G$1.VPH_POWER@3, U$1G$1.VPH_POWER@4, U$1G$1.VPH_POWER@5, U$1G$1.VPH_POWER@6, U$1G$1.VPH_POWER@7
- net USB_HS_ID: now also U13.G, U15.G
Other:
- note added: "Boot Settings"
- note added: "S1 - USB Boot"
- note added: "S2 - USB Device Mode"
- note added: "To Camera"
- note added: "To DSI Converter"
- moved on the sheet: C1, C50, C8, F2, J7, R1, R6, R8, U$2

Commit message: Added charger, more boot settings, more power supplies, and fingerprint sensor
Parts:
- removed U$2: MICROSD, glasses:MICROSD
- added C10, C11, C12, C13, C14, C15, C16, C17, C21, C23: 1uF, thanics-capacitor:CL05A105MP5NNNC
- added C18, C19, C20: 100nF, thanics-capacitor:CL05A104MP5NNNC
- added C22: 10uF, thanics-capacitor:GRM188R61A106KE69D
- added J2: DF30FC-30DS-0.4V, thanics-connector:DF30FC-30DS-0.4V
- added R17, R18, R19, R20, R23, R24, R25, R26, R27, R28: 10k, thanics-resistor:RC0402JR-0710KL
- added R21, R22: 5.1k, thanics-resistor:RMCF0603JT5K10
- added R29: 2k, thanics-resistor:RC0402FR-072KL
- added U16: SSM3J338RSOT-23F, glasses:SSM3J338RSOT-23F
- added U17: NX3020NAK, glasses:NX3020NAK
- added U18: 2.8, glasses:MIC5504-2.8
- added U19: TCR2EF15SOT-25, glasses:TCR2EF15SOT-25
- added U20: MICROSD, glasses:MICROSD
- added U21: MCP73833, glasses:MCP73833
- J1: value AXK724147G -> BM10NB(0.8)-16DS-0.4V(51); device glasses:AXK724147G -> thanics-connector:BM10NB(0.8)-16DS-0.4V(51)
Connections:
- new net !FINGER_RST: J1.10, R20.1, U$1G$1.GPIO22
- new net CAM1_PWDN: J2.12, U$1G$2.GPIO33
- new net CAM1_RST: J2.8, U$1G$1.GPIO28
- new net CAM1_XCLK: J2.23, U$1G$1.GPIO27
- new net CHARGER_VCC: C23.1, R17.2, U$1G$1.USB_VBUS, U14.D, U21.VDD
- new net CHARGE_STAT1: R27.1, U$1G$2.GPIO50, U21.STAT1
- new net CHARGE_STAT2: R28.1, U$1G$2.GPIO51, U21.STAT2
- new net DSI_EN: C21.1, R25.2, U7.EN
- new net FINGER_INT: J1.8, U$1G$1.GPIO23
- new net N$24: F2.2, R16.2, R19.1, U14.S, U16.D
- new net N$25: R18.2, U16.G, U17.S
- new net N$26: R14.2, U7.ADDR, U7.REFCLK
- new net N$27: R26.2, U21.THERM
- new net N$28: R29.2, U21.PROG
- new net N$29: C20.1, U1.REGOUT
- new net PM_RESIN_N: R24.1, U$1G$2.PM_RESIN_N
- new net SPI0_CLK: J1.16, U$1G$1.GPIO19
- new net SPI0_CS: J1.12, U$1G$1.GPIO18
- new net SPI0_MISO: J1.11, U$1G$1.GPIO17
- new net SPI0_MOSI: J1.15, U$1G$1.GPIO16
- net +1V8: now also C11.1, C13.1, C14.1, C17.1, C18.1, C19.1, J1.5, J1.7, J2.10, J2.2, J2.30, J2.6, R20.2, R21.2, R22.2, R24.2, R25.1, R27.2, R28.2, U1.AD0/SDO, U1.CS, U1.VDD, U1.VDDIO, U18.VOUT, U19.VOUT, U7.VCC; no longer R14.2
- net +3V3: now also C15.2, J1.6
- net +5V: now also U16.S, U17.D; no longer F2.2, R16.2, U14.S
- net GND: now also C10.2, C11.2, C12.2, C13.2, C14.2, C15.1, C16.2, C17.2, C18.2, C19.2, C20.2, C21.2, C22.2, C23.2, J1.13, J1.14, J1.3, J1.4, J1.9, J2.18, J2.21, J2.25, J2.26, J2.27, J2.29, J2.4, R14.1, R17.1, R18.1, R19.2, R23.1, R26.1, R29.1, U1.FSYNC, U1.GND, U18.GND, U19.GND, U20.VSS, U21.VSS, U7.GND; no longer U$2.VSS
- net I2C0_SCL: now also R22.1, U1.SCL/SCLK
- net I2C0_SDA: now also R21.1, U1.SDA/SDI
- net I2C2_SCL: now also J2.14
- net I2C2_SDA: now also J2.16
- net I2C3_SCL: now also U7.SCL
- net I2C3_SDA: now also U7.SDA
- net MIPI_CSI1_CLK_N: now also J2.13
- net MIPI_CSI1_CLK_P: now also J2.15
- net MIPI_CSI1_DATA0_N: now also J2.9
- net MIPI_CSI1_DATA0_P: now also J2.11
- net MIPI_CSI1_DATA1_N: now also J2.17
- net MIPI_CSI1_DATA1_P: now also J2.19
- net N$15: now also C16.1, U7.VCORE; no longer R14.1
- net P$1: now also C10.1, C12.1, U$1G$1.CDC_VDD_SPKDRV, U$1G$1.CDC_VDD_SPKDRV@1, U18.EN, U18.VIN, U19.CTL, U19.VIN
- net SDC2_CLK: now also U20.CLK; no longer U$2.CLK
- net SDC2_CMD: now also U20.CMD; no longer U$2.CMD
- net SDC2_DATA_0: now also U20.DAT0; no longer U$2.DAT0
- net SDC2_DATA_1: now also U20.DAT1; no longer U$2.DAT1
- net SDC2_DATA_2: now also U20.DAT2; no longer U$2.DAT2
- net SDC2_DATA_3: now also U20.CD/DAT3; no longer U$2.CD/DAT3
- net USB_HS_ID: now also R23.2, U17.G
- net VBATT_IN: now also C22.1, U21.VBAT
- net VREG_L11_SDC: now also U20.VDD; no longer U$2.VDD
Other:
- note added: "Connector for FPC1020AM"
- note added: "R29(2k) = 500mA charge current"
- note added: "S3 - Fastboot Mode"
- note added: "Setup for Normal Operation: ALL OFF"
- note added: "Setup for OS Install: S1 - OFF S2 - ON (Device Mode) S3 - ON (Fastboot Mode) *5 sec after power up, turn S3 OFF"
- moved on the sheet: C1, C3, C5, C50, C6, C8, F1, F2, J7, L1, R1, R11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

Commit message: Started PCB component placement, made a premium service DRC
Parts:
- added C24: 1uF, thanics-capacitor:CL05A105MP5NNNC
- added J3: S2B-XH-A(LF)(SN), thanics-connector:S2B-XH-A(LF)(SN)
- added R30, R31, R32, R33: 5.1k, thanics-resistor:RC0402JR-075K1L
- R12, R13, R21, R22: device thanics-resistor:RMCF0603JT5K10 -> thanics-resistor:RC0402JR-075K1L
Connections:
- new net !SHUTDOWN_LVDS: U11.SHTDN#
- new net +1V5: C13.1, J2.6, U19.VOUT
- new net +2V8: C11.1, J2.2, J2.30, U18.VOUT
- net +1V8: now also R30.2, R31.2, R32.2, R33.2; no longer C11.1, C13.1, J2.2, J2.30, J2.6, U18.VOUT, U19.VOUT
- net +3V3: now also C24.1, U11.VDD
- net GND: now also C24.2, J3.2, U11.GND, U11.MODE14, U11.SWAP
- net I2C2_SCL: now also R30.1
- net I2C2_SDA: now also R31.1
- net I2C3_SCL: now also R33.1
- net I2C3_SDA: now also R32.1
- net VBATT_IN: now also J3.1
Other:
- moved on the sheet: R11

Commit message: Added gesture board, more level shifting and light sensor
Parts:
- added C25, C27, C29, C30, C31: 1uF, thanics-capacitor:CL05A105MP5NNNC
- added C26, C28, C32: 100nF, thanics-capacitor:CL05A104MP5NNNC
- added J4: GRPB042MWCN-RC, thanics-connector:GRPB042MWCN-RC
- added R34, R35, R36: 470R, thanics-resistor:RC0402JR-07470RL
- added R37, R41, R42, R43, R44, R45, R46, R47, R48, R49, R50, R51: 10k, thanics-resistor:RC0402JR-0710KL
- added R38, R39, R40: 5.1k, thanics-resistor:RC0402JR-075K1L
- added U22, U24, U25: FXMA2104UMX, glasses:FXMA2104UMX
- added U23: NX3020NAK, glasses:NX3020NAK
- added U26: LTR-303ALS-01, glasses:LTR-303ALS-01
Connections:
- removed net !RST: R2.2, TP3.TP, U10.PB3
- removed net !SHUTDOWN_INT: U10.PA3
- removed net I2C_SCL_5V: U10.PA7
- removed net I2C_SDA_5V/TPIDATA: TP2.TP, U10.PB1
- new net !FINGER_INT_1V8: R48.1, U24.B0
- new net !FINGER_INT_5V: R46.1, U10.PB2, U24.A0
- new net !GESTURE_INT: R49.1, U$1G$2.GPIO69, U25.B2
- new net !GESTURE_INT_3V3: J4.7, U25.A2
- new net !LIGHT_INT: R50.1, U$1G$2.GPIO108, U25.B3
- new net !LIGHT_INT_3V3: R51.1, U25.A3, U26.INT
- new net !SHUTDOWN_INT_1V8: R43.1, U22.B3
- new net !SHUTDOWN_INT_5V: R41.1, U10.PA3, U22.A3
- new net !TOUCH_INT_1V8: U24.B1
- new net !TOUCH_INT_5V: R45.1, U10.PA5, U24.A1
- new net !TPI_RST_1V8: R42.1, U22.B0
- new net !TPI_RST_5V: R2.2, TP3.TP, U10.PB3, U22.A0
- new net EXT_PROG_EN: U$1G$2.GPIO120, U23.G
- new net I2C0_SCL_3V3: J4.2, U25.A1, U26.SCL
- new net I2C0_SCL_5V: R40.1, U10.PA7, U22.A1
- new net I2C0_SDA_3V3: J4.8, U25.A0, U26.SDA
- new net I2C0_SDA_5V/TPIDATA: R38.1, TP2.TP, U10.PB1, U22.A2
- new net LED_B: J4.4, U$1G$2.GPIO62
- new net LED_G: J4.3, U$1G$2.GPIO109
- new net LED_R: J4.5, U$1G$2.PM_MPP4
- new net N$30: R36.1, U8.CRX3
- new net N$31: R35.1, U8.CRX2
- new net N$32: R34.1, U8.CRX1
- new net N$33: R37.1, U22.OE, U23.D
- new net N$35: R44.1, U24.OE
- new net N$36: R47.1, U25.OE
- new net N$37: C27.1, C28.1, U8.VREG
- new net RX1: R34.2
- new net RX2: R35.2
- new net RX3: R36.2
- net !TOUCH_INT: now also R39.1, U$1G$2.GPIO21
- net +1V5: now also C30.1
- net +1V8: now also C25.1, C26.1, C29.1, R39.2, R42.2, R43.2, R48.2, R49.2, R50.2, U11.VDDIO, U22.VCCB, U24.VCCB, U25.VCCB, U8.VDDHI
- net +2V8: now also C31.1
- net +3V3: now also C32.1, J4.1, R47.2, R51.2, U25.VCCA, U26.VDD; no longer U8.VDDHI
- net +5V: now also R37.2, R38.2, R40.2, R41.2, R44.2, R45.2, R46.2, U22.VCCA, U24.VCCA
- net DSI_EN: now also U$1G$2.GPIO118
- net GND: now also C25.2, C26.2, C27.2, C28.2, C29.2, C30.2, C31.2, C32.2, J4.6, U22.GND, U23.S, U24.GND, U25.GND, U26.GND, U8.GND
- net I2C0_SCL: now also U22.B1, U25.B1, U8.SCL
- net I2C0_SDA: now also U22.B2, U25.B0, U8.SDA
Other:
- note added: "Level Shifting"
- moved on the sheet: C14, C15, C18, C19, C20, C22, C23, C6, J1, R11, R2, R20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

Commit message: Layout almost done
Parts:
- removed C16, C17, C21, C24: 1uF, thanics-capacitor:CL05A105MP5NNNC
- removed R14, R25: 10k, thanics-resistor:RC0402JR-0710KL
- removed U11: SN65LVDS822VQFN48, glasses:SN65LVDS822VQFN48
- removed U7: SN65DSI83PBGA-N64, glasses:SN65DSI83PBGA-N64
- added J10, J11, J5, J6, J8, J9: U.FL, thanics-connector:U.FL
- added R52: 10k, thanics-resistor:RC0402JR-0710KL
Connections:
- removed net !SHUTDOWN_LVDS: U11.SHTDN#
- removed net FINGER_INT: J1.8, U$1G$1.GPIO23
- removed net N$1: U11.A0P, U7.A_Y0P
- removed net N$10: U11.A3N, U7.A_Y3N
- removed net N$11: U11.CLKP, U7.A_CLKP
- removed net N$12: U11.CLKN, U7.A_CLKN
- removed net N$15: C16.1, U7.VCORE
- removed net N$26: R14.2, U7.ADDR, U7.REFCLK
- removed net N$3: U11.A0N, U7.A_Y0N
- removed net N$4: U11.A1P, U7.A_Y1P
- removed net N$5: U11.A1N, U7.A_Y1N
- removed net N$7: U11.A2P, U7.A_Y2P
- removed net N$8: U11.A2N, U7.A_Y2N
- removed net N$9: U11.A3P, U7.A_Y3P
- new net N$34: R52.1
- net !FINGER_INT_1V8: now also J1.8, U$1G$1.GPIO23
- net !TOUCH_INT: no longer U$1G$2.GPIO21
- net !TOUCH_INT_1V8: now also U$1G$2.GPIO21
- net !TOUCH_INT_5V: now also U10.PA4; no longer U10.PA5
- net !TPI_RST_1V8: now also U22.B1; no longer U22.B0
- net !TPI_RST_5V: now also U22.A1; no longer U22.A0
- net +1V8: now also R52.2; no longer C17.1, R25.1, U11.VDDIO, U7.VCC
- net +3V3: no longer C24.1, U11.VDD
- net BATT_CNTL: now also U10.PA5; no longer U10.PA4
- net DSI_EN: no longer C21.1, R25.2, U7.EN
- net GND: now also J10.GND@0, J10.GND@1, J11.GND@0, J11.GND@1, J5.GND@0, J5.GND@1, J6.GND@0, J6.GND@1, J8.GND@0, J8.GND@1, J9.GND@0, J9.GND@1; no longer C16.2, C17.2, C21.2, C24.2, R14.1, U11.GND, U11.MODE14, U11.SWAP, U7.GND
- net I2C0_SCL: now also U22.B0; no longer U22.B1
- net I2C0_SCL_5V: now also U22.A0; no longer U22.A1
- net I2C3_SCL: no longer U7.SCL
- net I2C3_SDA: no longer U7.SDA
- net LED_B: now also U$1G$2.PM_MPP3
- net LED_G: now also U$1G$2.PM_MPP2
- net MIPI_DSI0_CLK_N: now also J11.SIGNAL; no longer U7.DACN
- net MIPI_DSI0_CLK_P: now also J10.SIGNAL; no longer U7.DACP
- net MIPI_DSI0_DATA0_N: now also J6.SIGNAL; no longer U7.DA0N
- net MIPI_DSI0_DATA0_P: now also J5.SIGNAL; no longer U7.DA0P
- net MIPI_DSI0_DATA1_N: now also J9.SIGNAL; no longer U7.DA1N
- net MIPI_DSI0_DATA1_P: now also J8.SIGNAL; no longer U7.DA1P
- net MIPI_DSI0_DATA2_N: no longer U7.DA2N
- net MIPI_DSI0_DATA2_P: no longer U7.DA2P
- net MIPI_DSI0_DATA3_N: no longer U7.DA3N
- net MIPI_DSI0_DATA3_P: no longer U7.DA3P
Other:
- note added: "S3 - SD Boot"
- note added: "S4 - Fastboot Mode"
- note added: "Setup for Fastboot OS Install: S1 - OFF S2 - ON (Device Mode) S3 - OFF S4 - ON (Fastboot Mode) *5 sec after power up, turn S3 OFF"
- note added: "Setup for SD OS Install: S1 - OFF S2 - OFF S3 - ON (SD Boot) S4 - OFF"
- note removed: "Display"
- note removed: "S3 - Fastboot Mode"
- note removed: "Setup for OS Install: S1 - OFF S2 - ON (Device Mode) S3 - ON (Fastboot Mode) *5 sec after power up, turn S3 OFF"
- moved on the sheet: C1, C29, C30, C31, C50, F2, J2, J7, R1, R11, R12, R13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
