File: glassesBoard/glassesBoard.sch (EAGLE design)
At the start: 121 parts, among them J1 BM10NB(0.8)-16DS-0.4V(51), J10 U.FL, J11 U.FL, J2 DF30FC-30DS-0.4V, J3 S2B-XH-A(LF)(SN), J4 GRPB042MWCN-RC, J5 U.FL, J6 U.FL, J7 105450-0101, J8 U.FL, J9 U.FL, U10 ATTINY20-MMH, U12 NLAS2750, U13 NX3020NAK, U14 SSM3J338RSOT-23F, U15 NX3020NAK, U16 SSM3J338RSOT-23F, U17 NX3020NAK, U18 2.8, U19 TCR2EF15SOT-25, U2 TPS613222A, U20 MICROSD, U21 MCP73833, U22 FXMA2104UMX, U23 NX3020NAK, U24 FXMA2104UMX, U25 FXMA2104UMX, U26 LTR-303ALS-01, U3 1.8, U4 3.3, U5 SSM3J338RSOT-23F, U6 SSM3J338RSOT-23F, U8 IQS263BDFN10, U9 NX3020NAK

Commit message: Removed light sensor, added serial port pins, added touch panel connector, small schematic fixes
Parts:
- removed C32: 100nF, thanics-capacitor:CL05A104MP5NNNC
- removed J10, J11, J6, J8, J9: U.FL, thanics-connector:U.FL
- removed R50, R51: 10k, thanics-resistor:RC0402JR-0710KL
- removed U26: LTR-303ALS-01, glasses:LTR-303ALS-01
- added C16, C17, C21, C24: 1uF, thanics-capacitor:CL05A105MP5NNNC
- added JP1: (no value), pinhead:PINHD-1X3/90
- added R14, R25, R53: 10k, thanics-resistor:RC0402JR-0710KL
- added U11: SN65LVDS822VQFN48, glasses:SN65LVDS822VQFN48
- added U7: SN65DSI83-Q1S-PQFP-G64, glasses:SN65DSI83-Q1S-PQFP-G64
- J5: value U.FL -> 0787324001; device thanics-connector:U.FL -> thanics-connector:0787324001
Connections:
- removed net !LIGHT_INT: R50.1, U$1G$2.GPIO108, U25.B3
- removed net !LIGHT_INT_3V3: R51.1, U25.A3, U26.INT
- new net !SHUTDOWN_LVDS: U11.SHTDN#
- new net N$1: U11.A0P, U7.A_Y0P
- new net N$10: U11.A3N, U7.A_Y3N
- new net N$11: U11.CLKP, U7.A_CLKP
- new net N$12: U11.CLKN, U7.A_CLKN
- new net N$15: R53.2, U7.REFCLK
- new net N$26: C17.1, U7.VCORE
- new net N$3: U11.A0N, U7.A_Y0N
- new net N$39: R25.2, U7.ADDR
- new net N$4: U11.A1P, U7.A_Y1P
- new net N$5: U11.A1N, U7.A_Y1N
- new net N$7: U11.A2P, U7.A_Y2P
- new net N$8: U11.A2N, U7.A_Y2N
- new net N$9: U11.A3P, U7.A_Y3P
- new net TPICLK_1V8: U$1G$2.GPIO32, U24.B0
- new net UART1_RX: JP1.2, U$1G$1.GPIO5
- new net UART1_TX: JP1.1, U$1G$1.GPIO4
- net !FINGER_INT_1V8: now also U24.B1; no longer U24.B0
- net !FINGER_INT_5V: now also U24.A1; no longer U24.A0
- net !SHUTDOWN_INT_1V8: now also U$1G$2.GPIO36
- net !TOUCH_INT_1V8: now also U24.B2; no longer U24.B1
- net !TOUCH_INT_5V: now also U24.A2; no longer U24.A1
- net !TPI_RST_1V8: now also U$1G$2.GPIO34
- net +1V8: now also C16.1, R14.1, U11.VDDIO, U7.VCC; no longer R50.2
- net +3V3: now also C24.1, U11.VDD; no longer C32.1, R51.2, U26.VDD
- net DSI_EN: now also C21.1, R14.2, U7.EN
- net GND: now also C16.2, C17.2, C21.2, C24.2, J5.4, JP1.3, R25.1, R53.1, U11.GND, U11.MODE14, U11.SWAP, U7.GND; no longer C32.2, J10.GND@0, J10.GND@1, J11.GND@0, J11.GND@1, J5.GND@0, J5.GND@1, J6.GND@0, J6.GND@1, J8.GND@0, J8.GND@1, J9.GND@0, J9.GND@1, U26.GND
- net I2C0_SCL_3V3: no longer U26.SCL
- net I2C0_SDA_3V3: no longer U26.SDA
- net I2C3_SCL: now also U7.SCL
- net I2C3_SDA: now also U7.SDA
- net MIPI_DSI0_CLK_N: now also U7.DACN; no longer J11.SIGNAL
- net MIPI_DSI0_CLK_P: now also U7.DACP; no longer J10.SIGNAL
- net MIPI_DSI0_DATA0_N: now also U7.DA0N; no longer J6.SIGNAL
- net MIPI_DSI0_DATA0_P: now also U7.DA0P; no longer J5.SIGNAL
- net MIPI_DSI0_DATA1_N: now also U7.DA1N; no longer J9.SIGNAL
- net MIPI_DSI0_DATA1_P: now also U7.DA1P; no longer J8.SIGNAL
- net MIPI_DSI0_DATA2_N: now also U7.DA2N
- net MIPI_DSI0_DATA2_P: now also U7.DA2P
- net MIPI_DSI0_DATA3_N: now also U7.DA3N
- net MIPI_DSI0_DATA3_P: now also U7.DA3P
- net RX1: now also J5.2
- net RX2: now also J5.1
- net RX3: now also J5.3
- net TPICLK: now also U24.A0
Other:
- moved on the sheet: R46
