File: glassesBoard/glassesBoard.sch (EAGLE design)
At the start: 135 parts, among them J1 BM10NB(0.8)-16DS-0.4V(51), J2 DF30FC-30DS-0.4V, J3 S2B-XH-A(LF)(SN), J4 GRPB042MWCN-RC, J5 0787324001, J6 FH26W-39S-0.3SHW, J7 105450-0101, J8 5-520315-2, U10 ATTINY20-MMH, U11 SN65LVDS822VQFN48, U12 NLAS2750, U13 NX3020NAK, U14 SSM3J338RSOT-23F, U15 NX3020NAK, U16 SSM3J338RSOT-23F, U17 NX3020NAK, U18 2.8, U19 TCR2EF15SOT-25, U2 TPS613222A, U20 MICROSD, U21 MCP73833, U22 FXMA2104UMX, U23 NX3020NAK, U24 FXMA2104UMX, U25 FXMA2104UMX, U26 LM2665M6XSOT23-6, U27 NX3020NAK, U3 1.8, U4 3.3, U5 SSM3J338RSOT-23F, U6 SSM3J338RSOT-23F, U7 SN65DSI83-Q1S-PQFP-G64, U8 IQS263BDFN10, U9 NX3020NAK

Commit message: Fixed backwards display connector and changed backlight connector
Parts:
- removed C36: 1uF, thanics-capacitor:CL05A105MP5NNNC
- added R55, R56: 10k, thanics-resistor:RC0402JR-0710KL
- added R57, R58: 0R, thanics-resistor:RC0402JR-0710KL
- J8: value 5-520315-2 -> 62674-081121ALF; device thanics-connector:5-520315-2 -> thanics-connector:62674-081121ALF
- U17: value NX3020NAK -> SSM3J338RSOT-23F; device glasses:NX3020NAK -> glasses:SSM3J338RSOT-23F
Connections:
- new net N$45: R56.1, U10.PA1
- new net USB_POW: R16.1, R55.1, U14.G, U15.D, U17.G
- net +10V: now also J6.36; no longer J6.4
- net +1V8: now also J6.25, J6.9, R56.2; no longer J6.15, J6.31, U10.PA1
- net +3V3: now also J8.2, J8.3
- net +5V: now also R55.2, U17.S; no longer U17.D
- net B0: now also J6.2, U11.D8; no longer J6.38, U11.D12
- net B1: now also J6.3, U11.D7; no longer J6.37, U11.D13
- net B2: now also J6.4, U11.D6; no longer J6.36, U11.D14
- net B3: now also J6.5, U11.D22; no longer J6.35, U11.D15
- net B4: now also J6.6, U11.D21; no longer J6.34, U11.D16
- net B5: now also J6.7, U11.D5; no longer J6.33, U11.D17
- net B6: now also J6.10, U11.D4; no longer J6.30, U11.D25
- net B7: now also J6.11, U11.D3; no longer J6.29, U11.D26
- net CABC: now also J6.8; no longer J6.32
- net CLKX: now also J6.17; no longer J6.23
- net COM: now also J6.38; no longer J6.2
- net CSTN: now also J6.37; no longer J6.3
- net DE: now also J6.16, U11.D0; no longer J6.24, U11.D20
- net DSI_EN: now also R57.1, R58.1; no longer U11.SHTDN#, U7.EN
- net G0: now also J6.12, U11.D14; no longer J6.28, U11.D6
- net G1: now also J6.13, U11.D13; no longer J6.27, U11.D7
- net G2: now also J6.14, U11.D12; no longer J6.26, U11.D8
- net G3: now also J6.15, U11.D24; no longer J6.25, U11.D9
- net G4: now also J6.19, U11.D23; no longer J6.21, U11.D10
- net G6: now also J6.21, U11.D10; no longer J6.19, U11.D23
- net G7: now also J6.22, U11.D9; no longer J6.18, U11.D24
- net GND: now also C35.2, J6.18, J6.35; no longer C36.2, J6.22, J6.5
- net I2C0_SCL: now also J6.32; no longer J6.8
- net I2C0_SDA: now also J6.33; no longer J6.7
- net N$23: now also R57.2, U7.EN; no longer R16.1, U14.G, U15.D
- net N$25: now also U17.D; no longer U17.S
- net N$42: now also R58.2, U11.SHTDN#; no longer C35.2, C36.1
- net N$43: now also J8.6, J8.7, J8.8; no longer J8.2
- net R0: now also J6.23, U11.D20; no longer J6.17, U11.D0
- net R1: now also J6.24, U11.D19; no longer J6.16, U11.D1
- net R2: now also J6.26, U11.D18; no longer J6.14, U11.D2
- net R3: now also J6.27, U11.D26; no longer J6.13, U11.D3
- net R4: now also J6.28, U11.D25; no longer J6.12, U11.D4
- net R5: now also J6.29, U11.D17; no longer J6.11, U11.D5
- net R6: now also J6.30, U11.D16; no longer J6.10, U11.D21
- net R7: now also J6.31, U11.D15; no longer J6.9, U11.D22
- net RESETB: now also J6.34; no longer J6.6
- net TEST_HV: now also J6.39; no longer J6.1
- net USB_HS_ID: no longer U17.G
Other:
- note added: "Input Protection: U5 - Reverse polarity protection for battery F1 - 2A fuse (blows at 5A within 5 sec) FUSED_VBATT- ATTiny turns U6 OFF when ADC senses abnormal voltage drop across fuse F1"
- note added: "Power ON sequence: Touch Sensor reads button press, sends interrupt low, ATTiny turns U6 ON"
- note removed: "Input Protection: U5 - Reverse polarity protection for battery F1 - 2A fuse (blows at 5A within 5 sec) FUSE_SNS - ATTiny turns U6 OFF when ADC senses abnormal voltage drop across fuse F1"
- note removed: "Power ON sequence: Touch Sensor reads button press, sends interrupt low, U6 turns ON. ATTiny latches U6 ON before Touch interrupt goes high"
- moved on the sheet: C21, C32, C33, R14, R18, R4, R50, R51, R54, U27
