File: gestureBoard/gestureBoard.sch (EAGLE design)
At the start: 11 parts, among them J1 GRPB042MWCN-RC, U1 APDS-9960

Commit message: more progress on routing
Parts:
- added U3: PCA9553TSSOP8, glasses:PCA9553TSSOP8
Connections:
- net +3V3: now also U3.VDD
- net GND: now also U3.GND
- net LED_B: now also U3.LED2; no longer J1.4
- net LED_G: now also U3.LED1; no longer J1.3
- net LED_R: now also U3.LED0; no longer J1.5
- net SCL: now also U3.SCL
- net SDA: now also U3.SDA
Changed lines of the file:
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@@
 <part name="+3V4" library="supply1" deviceset="+3V3" device=""/>
 <part name="GND3" library="supply1" deviceset="GND" device=""/>
+<part name="U3" library="glasses" deviceset="PCA9553" device="TSSOP8" package3d_urn="urn:adsk.eagle:package:6948348/1"/>
+<part name="+3V5" library="supply1" deviceset="+3V3" device=""/>
+<part name="GND4" library="supply1" deviceset="GND" device=""/>
 </parts>
 <sheets>
@@
 <instance part="GND3" gate="1" x="60.96" y="-2.54" smashed="yes">
 <attribute name="VALUE" x="58.42" y="-5.08" size="1.778" layer="96"/>
+</instance>
+<instance part="U3" gate="G$1" x="27.94" y="-33.02" smashed="yes">
+<attribute name="NAME" x="20.32" y="-21.59" size="3.81" layer="95"/>
+</instance>
+<instance part="+3V5" gate="G$1" x="10.16" y="-20.32" smashed="yes" rot="MR0">
+<attribute name="VALUE" x="12.7" y="-25.4" size="1.778" layer="96" rot="MR90"/>
+</instance>
+<instance part="GND4" gate="1" x="12.7" y="-40.64" smashed="yes">
+<attribute name="VALUE" x="10.16" y="-43.18" size="1.778" layer="96"/>
 </instance>
 </instances>
@@
 <wire x1="5.08" y1="7.62" x2="5.08" y2="12.7" width="0.1524" layer="91"/>
 </segment>
+<segment>
+<pinref part="U3" gate="G$1" pin="VDD"/>
+<pinref part="+3V5" gate="G$1" pin="+3V3"/>
+<wire x1="15.24" y1="-27.94" x2="10.16" y2="-27.94" width="0.1524" layer="91"/>
+<wire x1="10.16" y1="-27.94" x2="10.16" y2="-22.86" width="0.1524" layer="91"/>
+</segment>
 </net>
 <net name="N$1" class="0">
@@
 </segment>
 <segment>
-<pinref part="J1" gate="G$1" pin="5"/>
-<wire x1="40.64" y1="0" x2="55.88" y2="0" width="0.1524" layer="91"/>
-<label x="43.18" y="0" size="1.778" layer="95"/>
+<pinref part="U3" gate="G$1" pin="LED0"/>
+<wire x1="40.64" y1="-27.94" x2="55.88" y2="-27.94" width="0.1524" layer="91"/>
+<label x="43.18" y="-27.94" size="1.778" layer="95"/>
 </segment>
 </net>
@@
 </segment>
 <segment>
-<pinref part="J1" gate="G$1" pin="3"/>
-<wire x1="20.32" y1="2.54" x2="5.08" y2="2.54" width="0.1524" layer="91"/>
-<label x="10.16" y="2.54" size="1.778" layer="95"/>
+<pinref part="U3" gate="G$1" pin="LED1"/>
+<wire x1="40.64" y1="-30.48" x2="55.88" y2="-30.48" width="0.1524" layer="91"/>
+<label x="43.18" y="-30.48" size="1.778" layer="95"/>
 </segment>
 </net>
@@
 </segment>
 <segment>
-<pinref part="J1" gate="G$1" pin="4"/>
-<wire x1="20.32" y1="0" x2="5.08" y2="0" width="0.1524" layer="91"/>
-<label x="10.16" y="0" size="1.778" layer="95"/>
+<pinref part="U3" gate="G$1" pin="LED2"/>
+<wire x1="40.64" y1="-33.02" x2="55.88" y2="-33.02" width="0.1524" layer="91"/>
+<label x="43.18" y="-33.02" size="1.778" layer="95"/>
 </segment>
 </net>
@@
 <wire x1="60.96" y1="2.54" x2="60.96" y2="0" width="0.1524" layer="91"/>
 </segment>
+<segment>
+<pinref part="U3" gate="G$1" pin="GND"/>
+<pinref part="GND4" gate="1" pin="GND"/>
+<wire x1="15.24" y1="-35.56" x2="12.7" y2="-35.56" width="0.1524" layer="91"/>
+<wire x1="12.7" y1="-35.56" x2="12.7" y2="-38.1" width="0.1524" layer="91"/>
+</segment>
 </net>
 <net name="N$4" class="0">
@@
 <label x="12.7" y="5.08" size="1.778" layer="95"/>
 </segment>
+<segment>
+<pinref part="U3" gate="G$1" pin="SCL"/>
+<wire x1="15.24" y1="-33.02" x2="5.08" y2="-33.02" width="0.1524" layer="91"/>
+<label x="7.62" y="-33.02" size="1.778" layer="95"/>
+</segment>
 </net>
 <net name="SDA" class="0">
@@
 <label x="43.18" y="7.62" size="1.778" layer="95"/>
 </segment>
+<segment>
+<pinref part="U3" gate="G$1" pin="SDA"/>
+<wire x1="15.24" y1="-30.48" x2="5.08" y2="-30.48" width="0.1524" layer="91"/>
+<label x="7.62" y="-30.48" size="1.778" layer="95"/>
+</segment>
 </net>
 </nets>
@@
 </schematic>
 </drawing>
+<compatibility>
+<note version="8.3" severity="warning">
+Since Version 8.3, EAGLE supports URNs for individual library
+assets (packages, symbols, and devices). The URNs of those assets
+will not be understood (or retained) with this version.
+</note>
+<note version="8.3" severity="warning">
+Since Version 8.3, EAGLE supports the association of 3D packages
+with devices in libraries, schematics, and board files. Those 3D
+packages will not be understood (or retained) with this version.
+</note>
+</compatibility>
 </eagle>
